Commit message: Moving head test

File: hrl4in/envs/gibson/jr2_kinova_head.urdf (robot description, URDF)
Before this commit: robot segway_robot, 39 links, 38 joints
Joints:
- joint pan_joint: type revolute -> fixed
- joint tilt_joint: limit lower=-0.261799 upper=0.261799 effort=60.0 velocity=6.597 -> lower=-0.52 upper=0.52 effort=60.0 velocity=6.597
